File: luca.sch (EAGLE design)
At the start: 60 parts

Commit message: fixed Jumper
Connections:
- removed net N$12: J1.1, MCU.PTE24
- net VDD: now also J1.1
Changed lines of the file:
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@@
 <label x="-43.18" y="27.94" size="1.27" layer="95" xref="yes"/>
+</segment>
+<segment>
+<pinref part="J1" gate="G$1" pin="1"/>
+<wire x1="111.76" y1="30.48" x2="111.76" y2="33.02" width="0.1524" layer="91"/>
+<label x="111.76" y="33.02" size="1.27" layer="95" rot="R90" xref="yes"/>
 </segment>
 </net>
@@
 </segment>
 </net>
-<net name="N$12" class="0">
-<segment>
-<pinref part="MCU" gate="A" pin="PTE24"/>
-<pinref part="J1" gate="G$1" pin="1"/>
-<wire x1="111.76" y1="30.48" x2="109.22" y2="30.48" width="0.1524" layer="91"/>
-</segment>
-</net>
